File: hardware/KiCAD/USB_VSense_gamma/USB_VSense_gamma.kicad_pcb (KiCad board)
At the start: 4 copper layers, 140.2 x 47.5 mm, 87 parts, among them J1 USB_C_Receptacle, J2 Conn_PIC_ICSP_ICD, P1 USB_C_Plug, U1 ATtiny406-M, U2 MCP1792x-5002xCB

Commit message: final changes
Other:
- board text added: "License: CERN-OHL-S-2.0"
Changed lines of the file:
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@@
 	)
 	(paper "A5")
+	(title_block
+		(title "USB VSense")
+		(date "28 January 2026")
+		(rev "Gamma")
+		(company "Meticulous Technologies")
+		(comment 1 "Copyright (C) 2026 Meticulous Technologies Licensed under CERN-OHL-S-2.0")
+	)
 	(layers
 		(0 "F.Cu" jumper)
@@
 			(size 3.5 3.5)
 			(drill 3.5)
-			(layers "F&B.Cu" "*.Mask")
+			(layers "*.Cu" "*.Mask")
 		)
 		(embedded_fonts no)
@@
 			(size 3.5 3.5)
 			(drill 3.5)
-			(layers "F&B.Cu" "*.Mask")
+			(layers "*.Cu" "*.Mask")
 		)
 		(embedded_fonts no)
@@
 			(size 1.8 1.8)
 			(drill 1.8)
-			(layers "F&B.Cu" "*.Mask")
+			(layers "*.Cu" "*.Mask")
 		)
 		(embedded_fonts no)
@@
 			(size 1.8 1.8)
 			(drill 1.8)
-			(layers "F&B.Cu" "*.Mask")
+			(layers "*.Cu" "*.Mask")
 		)
 		(embedded_fonts no)
@@
 			(size 3.5 3.5)
 			(drill 3.5)
-			(layers "F&B.Cu" "*.Mask")
+			(layers "*.Cu" "*.Mask")
 		)
 		(embedded_fonts no)
@@
 			(size 3.5 3.5)
 			(drill 3.5)
-			(layers "F&B.Cu" "*.Mask")
+			(layers "*.Cu" "*.Mask")
 		)
 		(embedded_fonts no)
@@
 			(size 5.58 5.58)
 			(drill 5.08)
-			(layers "F&B.Cu" "*.Mask")
+			(layers "*.Cu" "*.Mask")
 		)
 		(embedded_fonts no)
@@
 			(size 5.58 5.58)
 			(drill 5.08)
-			(layers "F&B.Cu" "*.Mask")
+			(layers "*.Cu" "*.Mask")
 		)
 		(embedded_fonts no)
@@
 			(size 1.8 1.8)
 			(drill 1.8)
-			(layers "F&B.Cu" "*.Mask")
+			(layers "*.Cu" "*.Mask")
 		)
 		(embedded_fonts no)
@@
 			(size 5.58 5.58)
 			(drill 5.08)
-			(layers "F&B.Cu" "*.Mask")
+			(layers "*.Cu" "*.Mask")
 		)
 		(embedded_fonts no)
@@
 			(size 1.8 1.8)
 			(drill 1.8)
-			(layers "F&B.Cu" "*.Mask")
+			(layers "*.Cu" "*.Mask")
 		)
 		(embedded_fonts no)
@@
 			(size 5.58 5.58)
 			(drill 5.08)
-			(layers "F&B.Cu" "*.Mask")
+			(layers "*.Cu" "*.Mask")
 		)
 		(embedded_fonts no)
@@
 			(size 1.8 1.8)
 			(drill 1.8)
-			(layers "F&B.Cu" "*.Mask")
+			(layers "*.Cu" "*.Mask")
 		)
 		(embedded_fonts no)
@@
 			(size 1.8 1.8)
 			(drill 1.8)
-			(layers "F&B.Cu" "*.Mask")
+			(layers "*.Cu" "*.Mask")
 		)
 		(embedded_fonts no)
@@
 			(size 5.58 5.58)
 			(drill 5.08)
-			(layers "F&B.Cu" "*.Mask")
+			(layers "*.Cu" "*.Mask")
 		)
 		(embedded_fonts no)
@@
 			(size 1.8 1.8)
 			(drill 1.8)
-			(layers "F&B.Cu" "*.Mask")
+			(layers "*.Cu" "*.Mask")
 		)
 		(embedded_fonts no)
@@
 			(size 5.58 5.58)
 			(drill 5.08)
-			(layers "F&B.Cu" "*.Mask")
+			(layers "*.Cu" "*.Mask")
 		)
 		(embedded_fonts no)
@@
 			(size 0.6 0.6)
 			(drill 0.6)
-			(layers "F&B.Cu" "*.Mask")
+			(layers "*.Cu" "*.Mask")
 		)
 		(pad "" smd rect
@@
 			(size 0.85 0.6)
 			(drill oval 0.85 0.6)
-			(layers "F&B.Cu" "*.Mask")
+			(layers "*.Cu" "*.Mask")
 		)
 		(pad "A1" smd rect
@@
 			(size 1.8 1.8)
 			(drill 1.8)
-			(layers "F&B.Cu" "*.Mask")
+			(layers "*.Cu" "*.Mask")
 		)
 		(embedded_fonts no)
@@
 			(size 1.8 1.8)
 			(drill 1.8)
-			(layers "F&B.Cu" "*.Mask")
+			(layers "*.Cu" "*.Mask")
 		)
 		(embedded_fonts no)
@@
 			(size 5.58 5.58)
 			(drill 5.08)
-			(layers "F&B.Cu" "*.Mask")
+			(layers "*.Cu" "*.Mask")
 		)
 		(embedded_fonts no)
@@
 			(size 5.58 5.58)
 			(drill 5.08)
-			(layers "F&B.Cu" "*.Mask")
+			(layers "*.Cu" "*.Mask")
 		)
 		(embedded_fonts no)
@@
 			(size 1.8 1.8)
 			(drill 1.8)
-			(layers "F&B.Cu" "*.Mask")
+			(layers "*.Cu" "*.Mask")
 		)
 		(embedded_fonts no)
@@
 			(size 5.58 5.58)
 			(drill 5.08)
-			(layers "F&B.Cu" "*.Mask")
+			(layers "*.Cu" "*.Mask")
 		)
 		(embedded_fonts no)
@@
 			(size 3.5 3.5)
 			(drill 3.5)
-			(layers "F&B.Cu" "*.Mask")
+			(layers "*.Cu" "*.Mask")
 		)
 		(embedded_fonts no)
@@
 			(size 1.8 1.8)
 			(drill 1.8)
-			(layers "F&B.Cu" "*.Mask")
+			(layers "*.Cu" "*.Mask")
 		)
 		(embedded_fonts no)
@@
 			(size 1.8 1.8)
 			(drill 1.8)
-			(layers "F&B.Cu" "*.Mask")
+			(layers "*.Cu" "*.Mask")
 		)
 		(embedded_fonts no)
@@
 			(size 3.5 3.5)
 			(drill 3.5)
-			(layers "F&B.Cu" "*.Mask")
+			(layers "*.Cu" "*.Mask")
 		)
 		(embedded_fonts no)
@@
 			(size 5.58 5.58)
 			(drill 5.08)
-			(layers "F&B.Cu" "*.Mask")
+			(layers "*.Cu" "*.Mask")
 		)
 		(embedded_fonts no)
@@
 			(size 1.8 1.8)
 			(drill 1.8)
-			(layers "F&B.Cu" "*.Mask")
+			(layers "*.Cu" "*.Mask")
 		)
 		(embedded_fonts no)
@@
 			(size 5.58 5.58)
 			(drill 5.08)
-			(layers "F&B.Cu" "*.Mask")
+			(layers "*.Cu" "*.Mask")
 		)
 		(embedded_fonts no)
@@
 			(size 1.8 1.8)
 			(drill 1.8)
-			(layers "F&B.Cu" "*.Mask")
+			(layers "*.Cu" "*.Mask")
 		)
 		(embedded_fonts no)
@@
 			(size 1.8 1.8)
 			(drill 1.8)
-			(layers "F&B.Cu" "*.Mask")
+			(layers "*.Cu" "*.Mask")
 		)
 		(embedded_fonts no)
@@
 			(size 3.5 3.5)
 			(drill 3.5)
-			(layers "F&B.Cu" "*.Mask")
+			(layers "*.Cu" "*.Mask")
 		)
 		(embedded_fonts no)
@@
 			(size 5.58 5.58)
 			(drill 5.08)
-			(layers "F&B.Cu" "*.Mask")
+			(layers "*.Cu" "*.Mask")
 		)
 		(embedded_fonts no)
@@
 			(size 1.8 1.8)
 			(drill 1.8)
-			(layers "F&B.Cu" "*.Mask")
+			(layers "*.Cu" "*.Mask")
 		)
 		(embedded_fonts no)
@@
 			(size 1.8 1.8)
 			(drill 1.8)
-			(layers "F&B.Cu" "*.Mask")
+			(layers "*.Cu" "*.Mask")
 		)
 		(embedded_fonts no)
@@
 			(size 0.6 1.6)
 			(drill oval 0.6 1.6)
-			(layers "F&B.Cu" "*.Mask")
+			(layers "*.Cu" "*.Mask")
 		)
 		(pad "" np_thru_hole oval
@@
 			(size 0.6 1.9)
 			(drill oval 0.6 1.9)
-			(layers "F&B.Cu" "*.Mask")
+			(layers "*.Cu" "*.Mask")
 		)
 		(pad "" np_thru_hole oval
@@
 			(size 0.6 1.6)
 			(drill oval 0.6 1.6)
-			(layers "F&B.Cu" "*.Mask")
+			(layers "*.Cu" "*.Mask")
 		)
 		(pad "" np_thru_hole oval
@@
 			(size 0.6 1.9)
 			(drill oval 0.6 1.9)
-			(layers "F&B.Cu" "*.Mask")
+			(layers "*.Cu" "*.Mask")
 		)
 		(embedded_fonts no)
@@
 			(size 5.58 5.58)
 			(drill 5.08)
-			(layers "F&B.Cu" "*.Mask")
+			(layers "*.Cu" "*.Mask")
 		)
 		(embedded_fonts no)
@@
 			(size 5.58 5.58)
 			(drill 5.08)
-			(layers "F&B.Cu" "*.Mask")
+			(layers "*.Cu" "*.Mask")
 		)
 		(embedded_fonts no)
@@
 			(size 5.58 5.58)
 			(drill 5.08)
-			(layers "F&B.Cu" "*.Mask")
+			(layers "*.Cu" "*.Mask")
 		)
 		(embedded_fonts no)
@@
 			(size 1.8 1.8)
 			(drill 1.8)
-			(layers "F&B.Cu" "*.Mask")
+			(layers "*.Cu" "*.Mask")
 		)
 		(embedded_fonts no)
@@
 			(size 5.58 5.58)
 			(drill 5.08)
-			(layers "F&B.Cu" "*.Mask")
+			(layers "*.Cu" "*.Mask")
 		)
 		(embedded_fonts no)
@@
 			(size 1.8 1.8)
 			(drill 1.8)
-			(layers "F&B.Cu" "*.Mask")
+			(layers "*.Cu" "*.Mask")
 		)
 		(embedded_fonts no)
@@
 			(size 1.8 1.8)
 			(drill 1.8)
-			(layers "F&B.Cu" "*.Mask")
+			(layers "*.Cu" "*.Mask")
 		)
 		(embedded_fonts no)
@@
 			(size 3.5 3.5)
 			(drill 3.5)
-			(layers "F&B.Cu" "*.Mask")
+			(layers "*.Cu" "*.Mask")
 		)
 		(embedded_fonts no)
@@
 		)
 	)
+	(gr_text "License: CERN-OHL-S-2.0"
+		(at 38.481 77.089 90)
+		(layer "F.SilkS")
+		(effects
+			(font
+				(size 1 1)
+				(thickness 0.15)
+			)
+			(justify left bottom)
+		)
+	)
 	(gr_text "A"
 		(at 109.855 64.772 0)
@@
 		)
 	)
+	(gr_text "License: CERN-OHL-S-2.0"
+		(at 138.811 77.089 90)
+		(layer "F.SilkS")
+		(effects
+			(font
+				(size 1 1)
+				(thickness 0.15)
+			)
+			(justify left bottom)
+		)
+	)
 	(gr_text "A"
 		(at 109.982 49.532 0)
@@
 		)
 	)
+	(gr_text "License: CERN-OHL-S-2.0"
+		(at 77.851 77.089 90)
+		(layer "F.SilkS")
+		(effects
+			(font
+				(size 1 1)
+				(thickness 0.15)
+			)
+			(justify left bottom)
+		)
+	)
+	(gr_text "License: CERN-OHL-S-2.0"
+		(at 98.171 77.089 90)
+		(layer "F.SilkS")
+		(effects
+			(font
+				(size 1 1)
+				(thickness 0.15)
+			)
+			(justify left bottom)
+		)
+	)
 	(gr_text "A"
 		(at 109.855 72.392 0)
@@
 		)
 	)
+	(gr_text "License: CERN-OHL-S-2.0"
+		(at 57.531 77.089 90)
+		(layer "F.SilkS")
+		(effects
+			(font
+				(size 1 1)
+				(thickness 0.15)
+			)
+			(justify left bottom)
+		)
+	)
 	(gr_text "T"
 		(at 112.522 53.213 0)
@@
 		)
 	)
+	(gr_text "License: CERN-OHL-S-2.0"
+		(at 118.491 77.089 90)
+		(layer "F.SilkS")
+		(effects
+			(font
+				(size 1 1)
+				(thickness 0.15)
+			)
+			(justify left bottom)
+		)
+	)
 	(gr_text "A"
 		(at 103.632 68.582 0)
@@
 		)
 	)
+	(gr_text "License: CERN-OHL-S-2.0"
+		(at 159.131 54.229 90)
+		(layer "B.SilkS")
+		(effects
+			(font
+				(size 1 1)
+				(thickness 0.15)
+			)
+			(justify left bottom mirror)
+		)
+	)
