File: hardware/KiCAD/USB_VSense_gamma/USB_VSense_gamma.kicad_sch (KiCad schematic)
At the start: 40 parts, among them J1 USB_C_Receptacle, J2 Conn_PIC_ICSP_ICD, P1 USB_C_Plug, U1 ATtiny406-M, U2 MCP1792x-5002xCB

Commit message: add firmware
Other:
- title: USB-C Voltage Indicator -> USB VSense
Changed lines of the file:
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@@
 	(paper "A4")
 	(title_block
-		(title "USB-C Voltage Indicator")
-		(date "12-June-2024")
-		(rev "Beta")
+		(title "USB VSense")
+		(date "28-January-2026")
+		(rev "Gamma")
 		(company "Meticulous Technologies")
 	)
